Commit message: Update test.urdf

File: test.urdf (robot description, URDF)
Before this commit: robot gcr3_618, 7 links, 6 joints
Links:
- link base_link: geometry collision mesh filename=https://raw.githubusercontent.com/Mediter14/duco_support/me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 scale=1000 1000 1000; visual mesh filename=https://raw.githubusercontent.com/Mediter14/duco_support/me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 scale=1000 1000 1000
- link link_1: geometry collision mesh filename=https://raw.githubusercontent.com/Mediter14/duco_support/me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 scale=1000 1000 1000; visual mesh filename=https://raw.githubusercontent.com/Mediter14/duco_support/me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 scale=1000 1000 1000
- link link_2: geometry collision mesh filename=https://raw.githubusercontent.com/Mediter14/duco_support/me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 scale=1000 1000 1000; visual mesh filename=https://raw.githubusercontent.com/Mediter14/duco_support/me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 scale=1000 1000 1000
- link link_3: geometry collision mesh filename=https://raw.githubusercontent.com/Mediter14/duco_support/me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 scale=1000 1000 1000; visual mesh filename=https://raw.githubusercontent.com/Mediter14/duco_support/me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 scale=1000 1000 1000
- link link_4: geometry collision mesh filename=https://raw.githubusercontent.com/Mediter14/duco_support/me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 scale=1000 1000 1000; visual mesh filename=https://raw.githubusercontent.com/Mediter14/duco_support/me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 scale=1000 1000 1000
- link link_5: geometry collision mesh filename=https://raw.githubusercontent.com/Mediter14/duco_support/me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 scale=1000 1000 1000; visual mesh filename=https://raw.githubusercontent.com/Mediter14/duco_support/me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 scale=1000 1000 1000
- link link_6: geometry collision mesh filename=https://raw.githubusercontent.com/Mediter14/duco_support/me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 scale=1000 1000 1000; visual mesh filename=https://raw.githubusercontent.com/Mediter14/duco_support/me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 scale=1000 1000 1000

Commit message: Update test.urdf

File: test.urdf (robot description, URDF)
Before this commit: robot gcr3_618, 7 links, 6 joints
Links:
- link base_link: geometry collision mesh filename=https://raw.githubusercontent.com/Mediter14/duco_urdf_demo/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 scale=1000 1000 1000; visual mesh filename=https://raw.githubusercontent.com/Mediter14/duco_urdf_demo/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 scale=1000 1000 1000
- link link_1: geometry collision mesh filename=https://raw.githubusercontent.com/Mediter14/duco_urdf_demo/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 scale=1000 1000 1000; visual mesh filename=https://raw.githubusercontent.com/Mediter14/duco_urdf_demo/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 scale=1000 1000 1000
- link link_2: geometry collision mesh filename=https://raw.githubusercontent.com/Mediter14/duco_urdf_demo/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 scale=1000 1000 1000; visual mesh filename=https://raw.githubusercontent.com/Mediter14/duco_urdf_demo/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 scale=1000 1000 1000
- link link_3: geometry collision mesh filename=https://raw.githubusercontent.com/Mediter14/duco_urdf_demo/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 scale=1000 1000 1000; visual mesh filename=https://raw.githubusercontent.com/Mediter14/duco_urdf_demo/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 scale=1000 1000 1000
- link link_4: geometry collision mesh filename=https://raw.githubusercontent.com/Mediter14/duco_urdf_demo/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 scale=1000 1000 1000; visual mesh filename=https://raw.githubusercontent.com/Mediter14/duco_urdf_demo/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 scale=1000 1000 1000
- link link_5: geometry collision mesh filename=https://raw.githubusercontent.com/Mediter14/duco_urdf_demo/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 scale=1000 1000 1000; visual mesh filename=https://raw.githubusercontent.com/Mediter14/duco_urdf_demo/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 scale=1000 1000 1000
- link link_6: geometry collision mesh filename=https://raw.githubusercontent.com/Mediter14/duco_urdf_demo/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 scale=1000 1000 1000; visual mesh filename=https://raw.githubusercontent.com/Mediter14/duco_urdf_demo/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 scale=1000 1000 1000

Commit message: Update test.urdf

File: test.urdf (robot description, URDF)
Before this commit: robot gcr3_618, 7 links, 6 joints
Links:
- link base_link: geometry collision mesh filename=https://raw.githubusercontent.com/Mediter14/duco_urdf_demo/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; visual mesh filename=https://raw.githubusercontent.com/Mediter14/duco_urdf_demo/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
- link link_1: geometry collision mesh filename=https://raw.githubusercontent.com/Mediter14/duco_urdf_demo/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; visual mesh filename=https://raw.githubusercontent.com/Mediter14/duco_urdf_demo/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
- link link_2: geometry collision mesh filename=https://raw.githubusercontent.com/Mediter14/duco_urdf_demo/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; visual mesh filename=https://raw.githubusercontent.com/Mediter14/duco_urdf_demo/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
- link link_3: geometry collision mesh filename=https://raw.githubusercontent.com/Mediter14/duco_urdf_demo/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; visual mesh filename=https://raw.githubusercontent.com/Mediter14/duco_urdf_demo/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
- link link_4: geometry collision mesh filename=https://raw.githubusercontent.com/Mediter14/duco_urdf_demo/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; visual mesh filename=https://raw.githubusercontent.com/Mediter14/duco_urdf_demo/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
- link link_5: geometry collision mesh filename=https://raw.githubusercontent.com/Mediter14/duco_urdf_demo/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; visual mesh filename=https://raw.githubusercontent.com/Mediter14/duco_urdf_demo/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
- link link_6: geometry collision mesh filename=https://raw.githubusercontent.com/Mediter14/duco_urdf_demo/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; visual mesh filename=https://raw.githubusercontent.com/Mediter14/duco_urdf_demo/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
